File: PCB_Files/Sensor_Integration_Board.kicad_sch (KiCad schematic)
At the start: 0 parts

Commit message: General schematic clean up and footprint allocation.
Changed lines of the file:
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@@
 	(paper "A4")
 	(sheet
-		(at 74.295 39.37)
-		(size 46.99 44.45)
+		(at 73.66 20.32)
+		(size 52.07 49.53)
 		(exclude_from_sim no)
 		(in_bom yes)
@@
 		)
 		(property "Sheetname" "MicroController"
-			(at 74.295 38.6584 0)
+			(at 73.66 19.6084 0)
 			(show_name no)
 			(do_not_autoplace no)
@@
 		)
 		(property "Sheetfile" "MCU_Schematic.kicad_sch"
-			(at 74.295 84.4046 0)
+			(at 73.66 70.4346 0)
 			(show_name no)
 			(do_not_autoplace no)
@@
 	)
 	(sheet
-		(at 17.78 80.645)
-		(size 33.655 29.845)
+		(at 128.27 20.32)
+		(size 46.99 49.53)
 		(exclude_from_sim no)
 		(in_bom yes)
@@
 		)
 		(property "Sheetname" "Motor_Controls"
-			(at 17.78 79.9334 0)
+			(at 128.27 19.6084 0)
 			(show_name no)
 			(do_not_autoplace no)
@@
 		)
 		(property "Sheetfile" "Motor_Controls.kicad_sch"
-			(at 17.78 111.0746 0)
+			(at 128.27 70.4346 0)
 			(show_name no)
 			(do_not_autoplace no)
@@
 	)
 	(sheet
-		(at 17.78 40.64)
-		(size 33.655 29.21)
+		(at 17.78 20.32)
+		(size 53.34 49.53)
 		(exclude_from_sim no)
 		(in_bom yes)
@@
 		)
 		(property "Sheetname" "Power_Delivery"
-			(at 17.78 39.9284 0)
+			(at 17.78 19.6084 0)
 			(show_name no)
 			(do_not_autoplace no)
